Commit message: add free friction of caster wheel

File: urdf/hbot.urdf.xacro (robot description, xacro)
@@ -105,4 +105,11 @@
     <origin xyz="${caster_xoff} 0.0 ${-wheel_zoff-wheel_radius+caster_radius}" rpy="0 0 0"/>
   </joint>
+  <gazebo reference="front_caster">
+    <mu1 value="0.001"/>
+    <mu2 value="0.001"/>
+    <kp value="1000000.0" />
+    <kd value="1.0" />
+    <material>Gazebo/Cyan</material>
+  </gazebo>
   <!-- Lidar -->
   <link name="laser">
