Commit message: feat(urdf): match the simulated model to the real robot
Keep the sim URDF/xacro in lock-step with the real robot so Gazebo exercises
the same frame layout and diff-drive geometry Nav2 / Cartographer see on
hardware (mirrors hbot_bringup/config/hbot.urdf, the URDF the Pi loads):

- base_footprint is identity with base_link (was a 0.0825 m Z offset); laser
  at xyz="0.08 0 0.14" rpy="0 0 0" (was xyz="0 0 0.075", yaw pi); add
  imu_link at the base origin.
- wheel_separation 0.17 -> 0.20 to match the driver wheel_track; wheel joints
  re-derived from wheel_separation / wheel_radius, base_link frame kept at
  ground level.
- body box height 0.12 -> 0.11 m, lifted to z in [0.02, 0.13] so its top
  clears the 0.14 m lidar scan plane (a full-height box poked through the
  horizontal scan and produced a phantom obstacle ring around the robot).
- lidar sensor aligned to the YDLidar X3 (0.12-12 m, 10 Hz, full 360 deg);
  add a Gazebo IMU sensor on imu_link publishing /imu.
- regenerate hbot.urdf / hbot.sdf (the committed hbot.sdf was a 0-byte file
  from a previously failed generator run).

Co-Authored-By: Claude Sonnet 5 <noreply@anthropic.com>

File: urdf/hbot.urdf (robot description, URDF)
Before this commit: robot hbot, 6 links, 5 joints
Links:
- added link imu_link
- link base_link: geometry collision box size=0.17 0.14 0.11; visual box size=0.17 0.14 0.11
Joints:
- added joint imu_joint: type fixed, parent base_link, child imu_link, origin xyz=0 0 0 rpy=0 0 0
- joint base_joint: origin xyz=0 0 0.0825 rpy=0 0 0 -> xyz=0 0 0 rpy=0 0 0
- joint front_caster_joint: origin xyz=0.07 0.0 -0.07250000000000001 rpy=0 0 0 -> xyz=0.07 0.0 0.01 rpy=0 0 0
- joint left_wheel_joint: origin xyz=-0.05 0.085 -0.05 rpy=0 0 0 -> xyz=-0.05 0.1 0.0325 rpy=0 0 0
- joint lidar_joint: origin xyz=0 0 0.075 rpy=0 0 3.14 -> xyz=0.08 0 0.14 rpy=0 0 0
- joint right_wheel_joint: origin xyz=-0.05 -0.085 -0.05 rpy=0 0 0 -> xyz=-0.05 -0.1 0.0325 rpy=0 0 0

File: urdf/hbot.urdf.xacro (robot description, xacro)
@@ -3,23 +3,53 @@
   <xacro:include filename="inertials.xacro" />
   <xacro:include filename="materials.xacro" />
-  <!-- Define some constants -->
-  <xacro:property name="base_width" value="0.14"/>
-  <xacro:property name="base_height" value="0.12"/>
+  <!-- ==========================================================================
+       Kinematic constants.
+       These are kept in sync with the *real* robot so the simulation exercises
+       the same frame layout and diff-drive geometry Nav2 / Cartographer see on
+       hardware:
+         - frame tree matches src/hbot_bringup/config/hbot.urdf (the URDF
+           robot_state_publisher loads on the Pi): base_footprint == base_link,
+           laser at (0.08, 0, 0.14), imu_link at the base origin.
+         - wheel_separation / wheel_diameter match the Yahboom driver params
+           in src/hbot_bringup/config/yahboom_driver_params.yaml
+           (wheel_track: 0.2, wheel_diameter: 0.065).
+       ========================================================================== -->
+  <!-- Body bounding box (X x Y x Z), used for visuals/collision/inertia only -
+       the real robot models base_link as a bare frame. base_height is kept a
+       touch under the real 0.12 m shell so the top of the box stays below the
+       lidar scan plane (lidar_zoff, 0.14 m) - otherwise the simulated lidar
+       rays sweeping past the rear/sides hit the robot's own collision box and
+       Nav2 sees a phantom obstacle ring ~0.16 m around the robot. On the real
+       robot the lidar puck simply sits proud of the shell and never sees it. -->
   <xacro:property name="base_length" value="0.17"/>
-  <xacro:property name="wheel_radius" value="0.0325"/>
-  <xacro:property name="wheel_width" value="0.025"/>
-  <xacro:property name="wheel_ygap" value="0.015"/>
-  <xacro:property name="wheel_zoff" value="0.05"/>
-  <xacro:property name="wheel_xoff" value="0.05"/>
+  <xacro:property name="base_width"  value="0.14"/>
+  <xacro:property name="base_height" value="0.11"/>
+  <!-- Drive wheels -->
+  <xacro:property name="wheel_radius"     value="0.0325"/>   <!-- 0.065 m diameter -->
+  <xacro:property name="wheel_width"      value="0.025"/>
+  <xacro:property name="wheel_separation" value="0.20"/>     <!-- driver wheel_track -->
+  <xacro:property name="wheel_xoff"       value="0.05"/>     <!-- wheels sit behind the body centre -->
+  <!-- Support caster -->
   <xacro:property name="caster_radius" value="0.01"/>
-  <xacro:property name="caster_xoff" value="0.07"/>
+  <xacro:property name="caster_xoff"   value="0.07"/>
+  <!-- Lidar mount, relative to base_link - matches config/hbot.urdf on the Pi -->
+  <xacro:property name="lidar_xoff" value="0.08"/>
+  <xacro:property name="lidar_zoff" value="0.14"/>
+  <!-- Body box centre height. The base_link frame itself stays coincident with
+       base_footprint (as on the real robot); only the visual/collision box is
+       lifted. Bottom sits at 0.02 m (clear of the ground plane, wheels/caster
+       carry the robot) and the top lands at base_shell_bottom + base_height =
+       0.13 m, just under the 0.14 m lidar plane. -->
+  <xacro:property name="base_shell_bottom" value="0.02"/>
+  <xacro:property name="base_zoff" value="${base_shell_bottom + base_height/2}"/>
   <link name="base_footprint"/>
   <joint name="base_joint" type="fixed">
     <parent link="base_footprint"/>
     <child link="base_link"/>
-    <origin xyz="0 0 ${(wheel_radius+wheel_zoff)}" rpy="0 0 0"/>
+    <origin xyz="0 0 0" rpy="0 0 0"/>
   </joint>
   <link name="base_link">
     <visual>
+      <origin xyz="0 0 ${base_zoff}" rpy="0 0 0"/>
       <geometry>
         <box size="${base_length} ${base_width} ${base_height}"/>
@@ -30,4 +60,5 @@
     </visual>
     <collision>
+      <origin xyz="0 0 ${base_zoff}" rpy="0 0 0"/>
       <geometry>
         <box size="${base_length} ${base_width} ${base_height}"/>
@@ -35,5 +66,5 @@
     </collision>
     <xacro:solid_cuboid_inertial
-      rpy="0 0 0" xyz="0 0 0" mass="0.5"
+      rpy="0 0 0" xyz="0 0 ${base_zoff}" mass="0.5"
       x="${base_length}" y="${base_width}" z="${base_height}"
     />
@@ -74,5 +105,5 @@
       <parent link="base_link"/>
       <child link="${prefix}_link"/>
-      <origin xyz="${x_reflect*wheel_xoff} ${y_reflect*(base_width/2+wheel_ygap)} ${-wheel_zoff}" rpy="0 0 0"/>
+      <origin xyz="${x_reflect*wheel_xoff} ${y_reflect*wheel_separation/2} ${wheel_radius}" rpy="0 0 0"/>
       <axis xyz="0 1 0"/>
     </joint>
@@ -103,5 +134,5 @@
     <parent link="base_link"/>
     <child link="front_caster"/>
-    <origin xyz="${caster_xoff} 0.0 ${-wheel_zoff-wheel_radius+caster_radius}" rpy="0 0 0"/>
+    <origin xyz="${caster_xoff} 0.0 ${caster_radius}" rpy="0 0 0"/>
   </joint>
   <gazebo reference="front_caster">
@@ -132,5 +163,5 @@
     <parent link="base_link"/>
     <child link="laser"/>
-    <origin xyz="0 0 ${base_height/2+0.015}" rpy="0 0 3.14"/>
+    <origin xyz="${lidar_xoff} 0 ${lidar_zoff}" rpy="0 0 0"/>
   </joint>
   <gazebo reference="laser">
@@ -138,4 +169,6 @@
       <always_on>true</always_on>
       <visualize>false</visualize>
+      <!-- YDLidar X3: ~10 Hz, 360 deg, ~0.12-12 m usable range
+           (see src/ydlidar_x3/.../params/ydlidar_x3.yaml) -->
       <update_rate>10</update_rate>
       <ray>
@@ -144,11 +177,11 @@
             <samples>360</samples>
             <resolution>1</resolution>
-            <min_angle>-3.14</min_angle>
-            <max_angle>3.14</max_angle>
+            <min_angle>-3.141592653589793</min_angle>
+            <max_angle>3.141592653589793</max_angle>
           </horizontal>
         </scan>
         <range>
-          <min>0.25</min>
-          <max>6.0</max>
+          <min>0.12</min>
+          <max>12.0</max>
           <resolution>0.02</resolution>
         </range>
@@ -171,4 +204,28 @@
     <material>Gazebo/Yellow</material>
   </gazebo>
+  <!-- IMU - frame matches config/hbot.urdf on the Pi. The EKF only runs on
+       hardware (base_bringup.launch.py); in sim the diff-drive plugin
+       publishes odom->base_footprint directly, but the sensor is kept so the
+       fused-odometry path can be exercised in sim if desired. -->
+  <link name="imu_link"/>
+  <joint name="imu_joint" type="fixed">
+    <parent link="base_link"/>
+    <child link="imu_link"/>
+    <origin xyz="0 0 0" rpy="0 0 0"/>
+  </joint>
+  <gazebo reference="imu_link">
+    <sensor name="imu_sensor" type="imu">
+      <always_on>true</always_on>
+      <update_rate>200</update_rate>
+      <visualize>false</visualize>
+      <plugin name="imu_plugin" filename="libgazebo_ros_imu_sensor.so">
+        <ros>
+          <remapping>~/out:=imu</remapping>
+        </ros>
+        <initial_orientation_as_reference>false</initial_orientation_as_reference>
+        <frame_name>imu_link</frame_name>
+      </plugin>
+    </sensor>
+  </gazebo>
   <gazebo>
     <plugin name="two_front_wheeled_diff_drive" filename="libgazebo_ros_diff_drive.so">
@@ -176,5 +233,5 @@
       <left_joint>left_wheel_joint</left_joint>
       <right_joint>right_wheel_joint</right_joint>
-      <wheel_separation>${base_width + 2 * wheel_ygap}</wheel_separation>
+      <wheel_separation>${wheel_separation}</wheel_separation>
       <wheel_diameter>${2 * wheel_radius}</wheel_diameter>
       <max_wheel_torque>20</max_wheel_torque>

Commit message: feat(urdf): build the HBOT model from the CAD meshes
Work from feat/cad-model, committed as the base for the description
restructure: prepare_meshes.py turns models/*.stl into link-frame meshes and
cad_params.xacro; hbot.urdf.xacro produces hbot.urdf (real, frames only) and
hbot_sim.urdf (sim:=true, full Gazebo model). See docs/cad_model.md.

Co-Authored-By: Claude Opus 5.5 <noreply@anthropic.com>

File: urdf/hbot.urdf (robot description, URDF)
Before this commit: robot hbot, 7 links, 6 joints
Links:
- removed link front_caster
- removed link left_wheel_link
- removed link right_wheel_link
- link base_link: mass 0.5 -> None; geometry 
- link laser: mass 0.001 -> None; geometry 
Joints:
- removed joint front_caster_joint
- removed joint left_wheel_joint
- removed joint right_wheel_joint
- joint lidar_joint: origin xyz=0.08 0 0.14 rpy=0 0 0 -> xyz=0.0425 0.0 0.1368 rpy=0 0 0

File: urdf/hbot.urdf.xacro (robot description, xacro)
@@ -1,46 +1,37 @@
 <?xml version="1.0" ?>
 <robot name="hbot" xmlns:xacro="http://ros.org/wiki/xacro">
-  <xacro:include filename="inertials.xacro" />
-  <xacro:include filename="materials.xacro" />
   <!-- ==========================================================================
-       Kinematic constants.
-       These are kept in sync with the *real* robot so the simulation exercises
-       the same frame layout and diff-drive geometry Nav2 / Cartographer see on
-       hardware:
-         - frame tree matches src/hbot_bringup/config/hbot.urdf (the URDF
-           robot_state_publisher loads on the Pi): base_footprint == base_link,
-           laser at (0.08, 0, 0.14), imu_link at the base origin.
-         - wheel_separation / wheel_diameter match the Yahboom driver params
-           in src/hbot_bringup/config/yahboom_driver_params.yaml
-           (wheel_track: 0.2, wheel_diameter: 0.065).
+       HBOT AMR - single source for both robot descriptions (see
+       docs/cad_model.md):
+         xacro hbot.urdf.xacro            -> hbot.urdf      real robot: TF frames
+                                                            only, for SLAM / Nav2
+         xacro hbot.urdf.xacro sim:=true  -> hbot_sim.urdf  Gazebo: + CAD meshes,
+                                                            collisions, inertias,
+                                                            wheels, caster, plugins
+       Frames (REP-103 / REP-105), identical in both:
+         base_footprint  on the ground, under the mid-point of the drive axle
+         base_link       coincident with base_footprint
+         laser           YDLidar X3 head centre, on the scan plane (the frame_id
+                         the ydlidar driver stamps on /scan)
+         imu_link        Rosmaster board IMU, at the base origin
+       x points forward (toward the caster), y left, z up.
        ========================================================================== -->
-  <!-- Body bounding box (X x Y x Z), used for visuals/collision/inertia only -
-       the real robot models base_link as a bare frame. base_height is kept a
-       touch under the real 0.12 m shell so the top of the box stays below the
-       lidar scan plane (lidar_zoff, 0.14 m) - otherwise the simulated lidar
-       rays sweeping past the rear/sides hit the robot's own collision box and
-       Nav2 sees a phantom obstacle ring ~0.16 m around the robot. On the real
-       robot the lidar puck simply sits proud of the shell and never sees it. -->
-  <xacro:property name="base_length" value="0.17"/>
-  <xacro:property name="base_width"  value="0.14"/>
-  <xacro:property name="base_height" value="0.11"/>
-  <!-- Drive wheels -->
-  <xacro:property name="wheel_radius"     value="0.0325"/>   <!-- 0.065 m diameter -->
-  <xacro:property name="wheel_width"      value="0.025"/>
-  <xacro:property name="wheel_separation" value="0.20"/>     <!-- driver wheel_track -->
-  <xacro:property name="wheel_xoff"       value="0.05"/>     <!-- wheels sit behind the body centre -->
-  <!-- Support caster -->
-  <xacro:property name="caster_radius" value="0.01"/>
-  <xacro:property name="caster_xoff"   value="0.07"/>
-  <!-- Lidar mount, relative to base_link - matches config/hbot.urdf on the Pi -->
-  <xacro:property name="lidar_xoff" value="0.08"/>
-  <xacro:property name="lidar_zoff" value="0.14"/>
-  <!-- Body box centre height. The base_link frame itself stays coincident with
-       base_footprint (as on the real robot); only the visual/collision box is
-       lifted. Bottom sits at 0.02 m (clear of the ground plane, wheels/caster
-       carry the robot) and the top lands at base_shell_bottom + base_height =
-       0.13 m, just under the 0.14 m lidar plane. -->
-  <xacro:property name="base_shell_bottom" value="0.02"/>
-  <xacro:property name="base_zoff" value="${base_shell_bottom + base_height/2}"/>
+  <xacro:arg name="sim" default="false"/>
+  <xacro:property name="sim" value="$(arg sim)"/>
+  <!-- Dimensions measured from the CAD (models/*.stl) by
+       scripts/prepare_meshes.py - regenerate, never hand-edit. -->
+  <xacro:include filename="cad_params.xacro" />
+  <!-- Drive wheels. The track is the real wheel_track (190-200 mm); the CAD
+       places the wheels at cad_wheel_separation (~183 mm). Keep this in sync
+       with wheel_track in hbot_bringup/config/yahboom_driver_params.yaml. -->
+  <xacro:property name="wheel_separation" value="0.195"/>
+  <xacro:property name="wheel_radius"     value="${cad_wheel_radius}"/>
+  <xacro:property name="wheel_width"      value="${cad_wheel_width}"/>
+  <xacro:if value="${sim}">
+    <xacro:include filename="inertials.xacro" />
+    <xacro:include filename="materials.xacro" />
+    <xacro:include filename="hbot_body.xacro" />
+  </xacro:if>
+  <!-- ===== Frames shared by the real robot and the simulation ===== -->
   <link name="base_footprint"/>
   <joint name="base_joint" type="fixed">
@@ -50,162 +41,14 @@
   </joint>
   <link name="base_link">
-    <visual>
-      <origin xyz="0 0 ${base_zoff}" rpy="0 0 0"/>
-      <geometry>
-        <box size="${base_length} ${base_width} ${base_height}"/>
-      </geometry>
-      <material name="Cyan">
-        <color rgba="0 1 1 1"/>
-      </material>
-    </visual>
-    <collision>
-      <origin xyz="0 0 ${base_zoff}" rpy="0 0 0"/>
-      <geometry>
-        <box size="${base_length} ${base_width} ${base_height}"/>
-      </geometry>
-    </collision>
-    <xacro:solid_cuboid_inertial
-      rpy="0 0 0" xyz="0 0 ${base_zoff}" mass="0.5"
-      x="${base_length}" y="${base_width}" z="${base_height}"
-    />
+    <xacro:if value="${sim}"><xacro:base_body/></xacro:if>
   </link>
-  <gazebo reference="base_link">
-    <material>Gazebo/Green</material>
-  </gazebo>
-  <!-- Wheel -->
-  <xacro:macro name="wheel" params="prefix x_reflect y_reflect">
-    <link name="${prefix}_link">
-      <visual>
-        <origin xyz="0 0 0" rpy="${pi/2} 0 0"/>
-        <geometry>
-          <cylinder radius="${wheel_radius}" length="${wheel_width}"/>
-          <cylinder radius="0.005" length="0.01">
-            <origin xyz="0 0 ${wheel_width/2+0.005}" rpy="0 0 0"/>
-          </cylinder>
-        </geometry>
-        <material name="Black">
-          <color rgba="0 0 0 1"/>
-        </material>
-      </visual>
-      <collision>
-        <origin xyz="0 0 0" rpy="${pi/2} 0 0"/>
-        <geometry>
-          <cylinder radius="${wheel_radius}" length="${wheel_width}"/>
-        </geometry>
-      </collision>
-      <xacro:solid_cylinder_inertial
-        rpy="0 0 0"
-        xyz="0 0 0"
-        mass="0.1"
-        radius="${wheel_radius}"
-        length="${wheel_width}"
-      />
-    </link>
-    <joint name="${prefix}_joint" type="continuous">
-      <parent link="base_link"/>
-      <child link="${prefix}_link"/>
-      <origin xyz="${x_reflect*wheel_xoff} ${y_reflect*wheel_separation/2} ${wheel_radius}" rpy="0 0 0"/>
-      <axis xyz="0 1 0"/>
-    </joint>
-    <gazebo reference="${prefix}_link">
-      <material>Gazebo/Black</material>
-    </gazebo>
-  </xacro:macro>
-  <xacro:wheel prefix="left_wheel" x_reflect="-1" y_reflect="1"/>
-  <xacro:wheel prefix="right_wheel" x_reflect="-1" y_reflect="-1"/>
-  <!-- Caster -->
-  <link name="front_caster">
-    <visual>
-      <geometry>
-        <sphere radius="${caster_radius}"/>
-      </geometry>
-      <material name="Cyan">
-        <color rgba="0 1.0 1.0 1.0"/>
-      </material>
-    </visual>
-    <collision>
-      <geometry>
-        <sphere radius="${caster_radius}"/>
-      </geometry>
-    </collision>
-    <xacro:null_inertial/>
-  </link>
-  <joint name="front_caster_joint" type="fixed">
-    <parent link="base_link"/>
-    <child link="front_caster"/>
-    <origin xyz="${caster_xoff} 0.0 ${caster_radius}" rpy="0 0 0"/>
-  </joint>
-  <gazebo reference="front_caster">
-    <mu1 value="0.001"/>
-    <mu2 value="0.001"/>
-    <kp value="1000000.0" />
-    <kd value="1.0" />
-    <material>Gazebo/Cyan</material>
-  </gazebo>
-  <!-- Lidar -->
   <link name="laser">
-    <visual>
-      <geometry>
-        <cylinder radius="0.03" length="0.025"/>
-      </geometry>
-      <material name="Gray">
-        <color rgba="0.5 0.5 0.5 1"/>
-      </material>
-    </visual>
-    <collision>
-      <geometry>
-        <cylinder radius="0.03" length="0.025"/>
-      </geometry>
-    </collision>
-    <xacro:null_inertial/>
+    <xacro:if value="${sim}"><xacro:lidar_body/></xacro:if>
   </link>
   <joint name="lidar_joint" type="fixed">
     <parent link="base_link"/>
     <child link="laser"/>
-    <origin xyz="${lidar_xoff} 0 ${lidar_zoff}" rpy="0 0 0"/>
+    <origin xyz="${cad_laser_x} ${cad_laser_y} ${cad_laser_z}" rpy="0 0 0"/>
   </joint>
-  <gazebo reference="laser">
-    <sensor name="lidar" type="ray">
-      <always_on>true</always_on>
-      <visualize>false</visualize>
-      <!-- YDLidar X3: ~10 Hz, 360 deg, ~0.12-12 m usable range
-           (see src/ydlidar_x3/.../params/ydlidar_x3.yaml) -->
-      <update_rate>10</update_rate>
-      <ray>
-        <scan>
-          <horizontal>
-            <samples>360</samples>
-            <resolution>1</resolution>
-            <min_angle>-3.141592653589793</min_angle>
-            <max_angle>3.141592653589793</max_angle>
-          </horizontal>
-        </scan>
-        <range>
-          <min>0.12</min>
-          <max>12.0</max>
-          <resolution>0.02</resolution>
-        </range>
-        <noise>
-          <type>gaussian</type>
-          <mean>0.0</mean>
-          <stddev>0.01</stddev>
-        </noise>
-      </ray>
-      <plugin name="scan" filename="libgazebo_ros_ray_sensor.so">
-        <ros>
-          <remapping>~/out:=scan</remapping>
-        </ros>
-        <output_type>sensor_msgs/LaserScan</output_type>
-        <frame_name>laser</frame_name>
-      </plugin>
-    </sensor>
-  </gazebo>
-  <gazebo reference="laser">
-    <material>Gazebo/Yellow</material>
-  </gazebo>
-  <!-- IMU - frame matches config/hbot.urdf on the Pi. The EKF only runs on
-       hardware (base_bringup.launch.py); in sim the diff-drive plugin
-       publishes odom->base_footprint directly, but the sensor is kept so the
-       fused-odometry path can be exercised in sim if desired. -->
   <link name="imu_link"/>
   <joint name="imu_joint" type="fixed">
@@ -214,36 +57,12 @@
     <origin xyz="0 0 0" rpy="0 0 0"/>
   </joint>
-  <gazebo reference="imu_link">
-    <sensor name="imu_sensor" type="imu">
-      <always_on>true</always_on>
-      <update_rate>200</update_rate>
-      <visualize>false</visualize>
-      <plugin name="imu_plugin" filename="libgazebo_ros_imu_sensor.so">
-        <ros>
-          <remapping>~/out:=imu</remapping>
-        </ros>
-        <initial_orientation_as_reference>false</initial_orientation_as_reference>
-        <frame_name>imu_link</frame_name>
-      </plugin>
-    </sensor>
-  </gazebo>
-  <gazebo>
-    <plugin name="two_front_wheeled_diff_drive" filename="libgazebo_ros_diff_drive.so">
-      <update_rate>30</update_rate>
-      <left_joint>left_wheel_joint</left_joint>
-      <right_joint>right_wheel_joint</right_joint>
-      <wheel_separation>${wheel_separation}</wheel_separation>
-      <wheel_diameter>${2 * wheel_radius}</wheel_diameter>
-      <max_wheel_torque>20</max_wheel_torque>
-      <max_wheel_acceleration>1.0</max_wheel_acceleration>
-      <command_topic>cmd_vel</command_topic>
-      <publish_odom>true</publish_odom>
-      <publish_odom_tf>true</publish_odom_tf>
-      <publish_wheel_tf>true</publish_wheel_tf>
-      <odometry_topic>odom</odometry_topic>
-      <odometry_frame>odom</odometry_frame>
-      <robot_base_frame>base_footprint</robot_base_frame>
-      <odometry_source>1</odometry_source>
-    </plugin>
-  </gazebo>
+  <!-- The real driver publishes no /joint_states, so the wheel joints stay
+       out of hbot.urdf - otherwise their TF would be missing on the robot. -->
+  <xacro:if value="${sim}">
+    <!-- ===== Simulation only ===== -->
+    <xacro:wheel prefix="left_wheel"  y_reflect="1"  mesh_yaw="0"/>
+    <xacro:wheel prefix="right_wheel" y_reflect="-1" mesh_yaw="${pi}"/>
+    <xacro:caster/>
+    <xacro:include filename="hbot.gazebo.xacro" />
+  </xacro:if>
 </robot>
