Commit message: refactor(description): one xacro + geometry YAML for real robot and Gazebo
Restructure hbot_description along common ROS 2 practice:

- config/hbot_geometry.yaml holds every dimension (wheel track now the
  measured 0.190 m; `cad` entries defer to cad_params.xacro), loaded with
  xacro.load_yaml().
- hbot.urdf.xacro is the single entry point (use_sim, driver_joint_states
  args); the model is split into hbot_base.xacro and hbot_sensors.xacro, with
  Gazebo tags only in hbot.gazebo.xacro. hbot_body.xacro is removed.
- The real robot now gets the full model (visuals, collisions, inertias);
  its wheels are fixed joints until the driver publishes /joint_states.
- hbot.urdf / hbot_sim.urdf / hbot_sim.sdf are generated into the build
  directory and installed (nothing written to src/, no longer tracked), so
  hbot_bringup and hbot_simulation keep working unchanged.
- New launch/description.launch.py (robot_state_publisher, xacro at launch)
  and launch/view.launch.py (+ joint_state_publisher + RViz);
  hbot_description.launch.py is kept as a deprecated wrapper.
- test/test_description.py: real/sim frame parity, wheel track vs. diff-drive
  and driver params, lidar spec, scan-plane clearance, meshes.
- docs/robot_description.md: step-by-step guide; cad_model.md trimmed to the
  CAD -> meshes part.

Co-Authored-By: Claude Opus 5.5 <noreply@anthropic.com>

File: urdf/hbot.gazebo.xacro (robot description, xacro)
@@ -1,6 +1,7 @@
 <?xml version="1.0" ?>
-<!-- Gazebo (classic) extensions for hbot.urdf.xacro: materials, contact
-     parameters, lidar + IMU sensors and the diff-drive plugin. Included from
-     hbot.urdf.xacro, which defines every property used here. -->
+<!-- Gazebo (classic) extensions: materials, contact parameters, lidar + IMU
+     sensor plugins and the diff-drive plugin. Included from hbot.urdf.xacro
+     only with use_sim:=true, which defines every property used here
+     (lidar specs: `lidar_sensor` in config/hbot_geometry.yaml). -->
 <robot xmlns:xacro="http://ros.org/wiki/xacro">
   <gazebo reference="base_link">
@@ -21,8 +22,5 @@
   <!-- YDLidar X3: 360 deg, 0.12-8 m, 3 kHz sampling at ~8 Hz scan rate
        -> 3000 / 8 = 375 samples per revolution. -->
-  <xacro:property name="lidar_rate"      value="8"/>
-  <xacro:property name="lidar_samples"   value="375"/>
-  <xacro:property name="lidar_range_min" value="0.12"/>
-  <xacro:property name="lidar_range_max" value="8.0"/>
+  <xacro:property name="lidar" value="${geo.lidar_sensor}"/>
   <gazebo reference="laser">
     <material>Gazebo/DarkGrey</material>
@@ -30,9 +28,9 @@
       <always_on>true</always_on>
       <visualize>false</visualize>
-      <update_rate>${lidar_rate}</update_rate>
+      <update_rate>${lidar.rate}</update_rate>
       <ray>
         <scan>
           <horizontal>
-            <samples>${lidar_samples}</samples>
+            <samples>${lidar.samples}</samples>
             <resolution>1</resolution>
             <min_angle>-3.141592653589793</min_angle>
@@ -41,6 +39,6 @@
         </scan>
         <range>
-          <min>${lidar_range_min}</min>
-          <max>${lidar_range_max}</max>
+          <min>${lidar.range_min}</min>
+          <max>${lidar.range_max}</max>
           <resolution>0.01</resolution>
         </range>
@@ -48,5 +46,5 @@
           <type>gaussian</type>
           <mean>0.0</mean>
-          <stddev>0.01</stddev>
+          <stddev>${lidar.noise_stddev}</stddev>
         </noise>
       </ray>

File: urdf/hbot.urdf.xacro (robot description, xacro)
@@ -2,67 +2,64 @@
 <robot name="hbot" xmlns:xacro="http://ros.org/wiki/xacro">
   <!-- ==========================================================================
-       HBOT AMR - single source for both robot descriptions (see
-       docs/cad_model.md):
-         xacro hbot.urdf.xacro            -> hbot.urdf      real robot: TF frames
-                                                            only, for SLAM / Nav2
-         xacro hbot.urdf.xacro sim:=true  -> hbot_sim.urdf  Gazebo: + CAD meshes,
-                                                            collisions, inertias,
-                                                            wheels, caster, plugins
-       Frames (REP-103 / REP-105), identical in both:
+       HBOT AMR - the single entry point of the robot description
+       (docs/robot_description.md):
+         xacro hbot.urdf.xacro                -> real robot (robot_state_publisher
+                                                 on the Pi, SLAM / Nav2 / RViz)
+         xacro hbot.urdf.xacro use_sim:=true  -> Gazebo model (+ sensors,
+                                                 diff-drive plugin, friction)
+       Both variants contain the same links, joints, visuals, collisions and
+       inertias; use_sim only adds the <gazebo> extensions. Every dimension
+       comes from config/hbot_geometry.yaml (which may defer to the CAD values
+       in cad_params.xacro) - no robot dimension is typed into the xacro files.
+       Frames (REP-103 / REP-105):
          base_footprint  on the ground, under the mid-point of the drive axle
          base_link       coincident with base_footprint
+         left/right_wheel_link, front_caster
          laser           YDLidar X3 head centre, on the scan plane (the frame_id
                          the ydlidar driver stamps on /scan)
-         imu_link        Rosmaster board IMU, at the base origin
+         imu_link        Rosmaster board IMU
        x points forward (toward the caster), y left, z up.
        ========================================================================== -->
-  <xacro:arg name="sim" default="false"/>
-  <xacro:property name="sim" value="$(arg sim)"/>
-  <!-- Dimensions measured from the CAD (models/*.stl) by
-       scripts/prepare_meshes.py - regenerate, never hand-edit. -->
-  <xacro:include filename="cad_params.xacro" />
-  <!-- Drive wheels. The track is the real wheel_track (190-200 mm); the CAD
-       places the wheels at cad_wheel_separation (~183 mm). Keep this in sync
-       with wheel_track in hbot_bringup/config/yahboom_driver_params.yaml. -->
-  <xacro:property name="wheel_separation" value="0.195"/>
-  <xacro:property name="wheel_radius"     value="${cad_wheel_radius}"/>
-  <xacro:property name="wheel_width"      value="${cad_wheel_width}"/>
-  <xacro:if value="${sim}">
-    <xacro:include filename="inertials.xacro" />
-    <xacro:include filename="materials.xacro" />
-    <xacro:include filename="hbot_body.xacro" />
-  </xacro:if>
-  <!-- ===== Frames shared by the real robot and the simulation ===== -->
-  <link name="base_footprint"/>
-  <joint name="base_joint" type="fixed">
-    <parent link="base_footprint"/>
-    <child link="base_link"/>
-    <origin xyz="0 0 0" rpy="0 0 0"/>
-  </joint>
-  <link name="base_link">
-    <xacro:if value="${sim}"><xacro:base_body/></xacro:if>
-  </link>
-  <link name="laser">
-    <xacro:if value="${sim}"><xacro:lidar_body/></xacro:if>
-  </link>
-  <joint name="lidar_joint" type="fixed">
-    <parent link="base_link"/>
-    <child link="laser"/>
-    <origin xyz="${cad_laser_x} ${cad_laser_y} ${cad_laser_z}" rpy="0 0 0"/>
-  </joint>
-  <link name="imu_link"/>
-  <joint name="imu_joint" type="fixed">
-    <parent link="base_link"/>
-    <child link="imu_link"/>
-    <origin xyz="0 0 0" rpy="0 0 0"/>
-  </joint>
-  <!-- The real driver publishes no /joint_states, so the wheel joints stay
-       out of hbot.urdf - otherwise their TF would be missing on the robot. -->
-  <xacro:if value="${sim}">
-    <!-- ===== Simulation only ===== -->
-    <xacro:wheel prefix="left_wheel"  y_reflect="1"  mesh_yaw="0"/>
-    <xacro:wheel prefix="right_wheel" y_reflect="-1" mesh_yaw="${pi}"/>
-    <xacro:caster/>
-    <xacro:include filename="hbot.gazebo.xacro" />
+  <!-- ===== Arguments ===== -->
+  <xacro:arg name="use_sim" default="false"/>
+  <!-- The real driver does not publish /joint_states yet, so on the real robot
+       the wheels are fixed joints (robot_state_publisher then publishes their
+       TF itself). Set true once hbot_driver publishes the wheel joint states. -->
+  <xacro:arg name="driver_joint_states" default="false"/>
+  <!-- xacro args are strings ("false" is truthy in Python): convert once here. -->
+  <xacro:property name="use_sim" value="${'$(arg use_sim)'.lower() in ('true', '1')}"/>
+  <xacro:property name="driver_joint_states" value="${'$(arg driver_joint_states)'.lower() in ('true', '1')}"/>
+  <!-- ===== Parameters ===== -->
+  <!-- CAD measurements (generated by scripts/prepare_meshes.py - never edit) -->
+  <xacro:include filename="cad_params.xacro"/>
+  <!-- Robot geometry (edit this one). The path is relative to this file, so it
+       works from the source tree and from the install space alike. -->
+  <xacro:property name="geo" value="${xacro.load_yaml('../config/hbot_geometry.yaml')}" lazy_eval="false"/>
+  <!-- Resolve `cad` entries of the YAML to the measured CAD values. -->
+  <xacro:property name="wheel_separation" value="${cad_wheel_separation if geo.wheels.track  == 'cad' else geo.wheels.track}"/>
+  <xacro:property name="wheel_radius"     value="${cad_wheel_radius     if geo.wheels.radius == 'cad' else geo.wheels.radius}"/>
+  <xacro:property name="wheel_width"      value="${cad_wheel_width      if geo.wheels.width  == 'cad' else geo.wheels.width}"/>
+  <xacro:property name="caster_x"         value="${cad_caster_x         if geo.caster.x      == 'cad' else geo.caster.x}"/>
+  <xacro:property name="caster_y"         value="${cad_caster_y         if geo.caster.y      == 'cad' else geo.caster.y}"/>
+  <xacro:property name="caster_radius"    value="${cad_caster_radius    if geo.caster.radius == 'cad' else geo.caster.radius}"/>
+  <xacro:property name="laser_x"          value="${cad_laser_x          if geo.laser.x       == 'cad' else geo.laser.x}"/>
+  <xacro:property name="laser_y"          value="${cad_laser_y          if geo.laser.y       == 'cad' else geo.laser.y}"/>
+  <xacro:property name="laser_z"          value="${cad_laser_z          if geo.laser.z       == 'cad' else geo.laser.z}"/>
+  <xacro:property name="laser_yaw"        value="${geo.laser.yaw}"/>
+  <xacro:property name="wheel_joint_type" value="${'continuous' if (use_sim or driver_joint_states) else 'fixed'}"/>
+  <!-- ===== Model ===== -->
+  <xacro:include filename="materials.xacro"/>
+  <xacro:include filename="inertials.xacro"/>
+  <xacro:include filename="hbot_base.xacro"/>
+  <xacro:include filename="hbot_sensors.xacro"/>
+  <xacro:hbot_base/>
+  <xacro:wheel prefix="left_wheel"  y_reflect="1"  mesh_yaw="0"/>
+  <xacro:wheel prefix="right_wheel" y_reflect="-1" mesh_yaw="${pi}"/>
+  <xacro:caster/>
+  <xacro:laser_sensor/>
+  <xacro:imu_sensor/>
+  <!-- ===== Simulation only ===== -->
+  <xacro:if value="${use_sim}">
+    <xacro:include filename="hbot.gazebo.xacro"/>
   </xacro:if>
 </robot>

Commit message: feat(urdf): blue base_link in Gazebo and RViz
hbot.gazebo.xacro: base_link Gazebo/Grey -> Gazebo/Blue; hbot_base.xacro:
base_link visual material gray -> blue so RViz matches. Guide: how to
change a part's colour.

Co-Authored-By: Claude Opus 5.5 <noreply@anthropic.com>

File: urdf/hbot.gazebo.xacro (robot description, xacro)
@@ -6,5 +6,5 @@
 <robot xmlns:xacro="http://ros.org/wiki/xacro">
   <gazebo reference="base_link">
-    <material>Gazebo/Grey</material>
+    <material>Gazebo/Blue</material>
   </gazebo>
   <gazebo reference="left_wheel_link">

File: urdf/hbot_base.xacro (robot description, xacro)
@@ -27,5 +27,5 @@
           <mesh filename="package://hbot_description/meshes/base_link.stl"/>
         </geometry>
-        <material name="gray"/>
+        <material name="blue"/>
       </visual>
       <collision>
